File: PCB/hackathon-badge.kicad_sch (KiCad schematic)
At the start: 0 parts

Commit message: update
Parts:
- added TP1, TP2, TP3, TP4: TestPoint, symbol Connector:TestPoint
Connections:
- new net GND: TP1.1, TP2.1, TP3.1, TP4.1
