File: OUTER_PCB/hackathon-badge.kicad_sch (KiCad schematic)
At the start: 18 parts

Commit message: finished the outer board
Parts:
- removed D15, D16, D17, D18: WS2812B-2020, LED_SMD:LED_WS2812B-2020_PLCC4_2.0x2.0mm, symbol LED:WS2812B-2020
- added TP1, TP2, TP3, TP4: TestPoint, TestPoint:TestPoint_Pad_4.0x4.0mm, symbol Connector:TestPoint
Connections:
- net +5V: now also TP2.1
- net GND: now also TP1.1, TP4.1
- net LED_DIN: now also TP3.1
Other:
- moved on the sheet: D1, D10, D11, D12, D13, D14, D2, D3, D4, D5, D6, D7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

Commit message: finished second PCB
Connections:
- net +5V renamed +3.7V
