File: INNER_PCB/INNER_PCB.kicad_pcb (KiCad board)
At the start: 2 copper layers, 50 x 50 mm, 10 parts, among them J1 Conn_01x03, J2 Conn_01x02, U2 CH32V003FxUx

Commit message: added the second side to the second PCB
Parts:
- added TP5: TestPoint, TestPoint:TestPoint_Pad_3.0x3.0mm, B.Cu at (144.2, 73.2)
- added TP6: TestPoint, TestPoint:TestPoint_Pad_3.0x3.0mm, B.Cu at (144.2, 120.2)
- added TP7: TestPoint, TestPoint:TestPoint_Pad_3.0x3.0mm, B.Cu at (120.7, 96.7)
- added TP8: TestPoint, TestPoint:TestPoint_Pad_3.0x3.0mm, B.Cu at (167.7, 96.7)
Routing:
- net /LED_DOUT: track 17.2 -> 54.6 mm
- net GND: track 1.61 -> 10.3 mm, vias 9 -> 10
- net +3.7V: vias 0 -> 1

Commit message: some more art for the inner badge
Parts:
- added G***: LOGO, LOGO, F.Cu at (139.4, 111.1)
- added G***: LOGO, LOGO, F.Cu at (133.8, 84.7)
- added G***: LOGO, LOGO, F.Cu at (155.8, 112.3)
- added G***: LOGO, LOGO, F.Cu at (157.5, 92.2)
- added G***: LOGO, LOGO, F.Cu at (151.7, 83.1)
- added G***: LOGO, LOGO, F.Cu at (154.2, 96.0)
- added G***: LOGO, LOGO, F.Cu at (129.2, 90.8)
- added G***: LOGO, LOGO, F.Cu at (154.5, 84.7)
- added G***: LOGO, LOGO, F.Cu at (147.6, 107.9)
- added G***: LOGO, LOGO, F.Cu at (154.3, 111.2)
- added G***: LOGO, LOGO, F.Cu at (135.4, 109.2)
- added G***: LOGO, LOGO, F.Cu at (130.4, 94.3)
- added G***: LOGO, LOGO, F.Cu at (152.2, 98.8)
- added G***: LOGO, LOGO, F.Cu at (137.1, 107.6)
- added G***: LOGO, LOGO, F.Cu at (131.9, 91.9)
Routing:
- net +3.7V: track 86.4 -> 84.7 mm

Commit message: update
Parts:
- added D1: KT-0603Y, LED_SMD:LED_0603_1608Metric, F.Cu at (129.4, 91.3)
- added D10: KT-0603Y, LED_SMD:LED_0603_1608Metric, B.Cu at (139.1, 110.4)
- added D11: KT-0603Y, LED_SMD:LED_0603_1608Metric, B.Cu at (144.2, 98.1)
- added D12: KT-0603Y, LED_SMD:LED_0603_1608Metric, B.Cu at (161.2, 100.9)
- added D13: KT-0603Y, LED_SMD:LED_0603_1608Metric, B.Cu at (130.7, 92.8)
- added D14: KT-0603Y, LED_SMD:LED_0603_1608Metric, B.Cu at (131.0, 98.5)
- added D15: KT-0603Y, LED_SMD:LED_0603_1608Metric, B.Cu at (134.7, 83.0)
- added D16: KT-0603Y, LED_SMD:LED_0603_1608Metric, B.Cu at (150.9, 82.6)
- added D2: KT-0603Y, LED_SMD:LED_0603_1608Metric, F.Cu at (151.6, 81.0)
- added D3: KT-0603Y, LED_SMD:LED_0603_1608Metric, F.Cu at (156.5, 89.2)
- added D4: KT-0603Y, LED_SMD:LED_0603_1608Metric, F.Cu at (127.7, 94.7)
- added D5: KT-0603Y, LED_SMD:LED_0603_1608Metric, F.Cu at (135.3, 111.2)
- added D6: KT-0603Y, LED_SMD:LED_0603_1608Metric, F.Cu at (146.8, 111.4)
- added D7: KT-0603Y, LED_SMD:LED_0603_1608Metric, F.Cu at (154.3, 94.1)
- added D8: KT-0603Y, LED_SMD:LED_0603_1608Metric, F.Cu at (138.6, 81.6)
- added D9: KT-0603Y, LED_SMD:LED_0603_1608Metric, F.Cu at (139.3, 99.8)
- added G***: LOGO, LOGO, B.Cu at (160.6, 102.8)
- added G***: LOGO, LOGO, B.Cu at (128.2, 99.1)
- added G***: LOGO, LOGO, B.Cu at (140.8, 79.5)
- added G***: LOGO, LOGO, B.Cu at (142.7, 94.6)
- added G***: LOGO, LOGO, B.Cu at (134.8, 95.9)
- added G***: LOGO, LOGO, B.Cu at (141.5, 112.4)
- added G***: LOGO, LOGO, B.Cu at (144.7, 97.1)
- added G***: LOGO, LOGO, B.Cu at (136.9, 95.1)
- added G***: LOGO, LOGO, B.Cu at (151.0, 84.7)
- added G***: LOGO, LOGO, B.Cu at (144.5, 100.8)
- added G***: LOGO, LOGO, B.Cu at (133.5, 85.4)
- added R10: 2k, Resistor_SMD:R_0402_1005Metric, F.Cu at (139.5, 101.1)
- added R11: 2k, Resistor_SMD:R_0402_1005Metric, B.Cu at (138.9, 111.6)
- added R12: 2k, Resistor_SMD:R_0402_1005Metric, B.Cu at (144.5, 96.8)
- added R13: 2k, Resistor_SMD:R_0402_1005Metric, B.Cu at (161.3, 99.6)
- added R14: 2k, Resistor_SMD:R_0402_1005Metric, B.Cu at (131.0, 91.5)
- added R15: 2k, Resistor_SMD:R_0402_1005Metric, B.Cu at (131.2, 97.1)
- added R16: 2k, Resistor_SMD:R_0402_1005Metric, B.Cu at (134.9, 81.8)
- added R17: 2k, Resistor_SMD:R_0402_1005Metric, B.Cu at (151.1, 81.3)
- added R2: 2k, Resistor_SMD:R_0402_1005Metric, F.Cu at (126.4, 91.4)
- added R3: 2k, Resistor_SMD:R_0402_1005Metric, F.Cu at (153.8, 81.3)
- added R4: 2k, Resistor_SMD:R_0402_1005Metric, F.Cu at (156.4, 90.6)
- added R5: 2k, Resistor_SMD:R_0402_1005Metric, F.Cu at (127.8, 96.1)
- added R6: 2k, Resistor_SMD:R_0402_1005Metric, F.Cu at (136.0, 112.6)
- added R7: 2k, Resistor_SMD:R_0402_1005Metric, F.Cu at (146.9, 112.8)
- added R8: 2k, Resistor_SMD:R_0402_1005Metric, F.Cu at (156.6, 95.5)
- added R9: 2k, Resistor_SMD:R_0402_1005Metric, F.Cu at (138.6, 83.1)
- moved G*** 0.32 mm to (135.3, 108.9)
Routing:
- net +3.7V: track 84.7 -> 175.7 mm, vias 1 -> 8
- net /LED_DOUT: track 54.6 -> 67.7 mm
- net Net-(D1-A): track 0.00 -> 4.25 mm
- net Net-(D7-A): track 0.00 -> 1.89 mm
- net Net-(D16-A): track 0.00 -> 1.75 mm
- net Net-(D15-A): track 0.00 -> 1.65 mm
- net Net-(D5-A): track 0.00 -> 1.64 mm
- net Net-(D8-A): track 0.00 -> 1.61 mm
- net Net-(D3-A): track 0.00 -> 1.55 mm
- net Net-(D2-A): track 0.00 -> 1.50 mm
- net Net-(D4-A): track 0.00 -> 1.47 mm
- net Net-(D6-A): track 0.00 -> 1.47 mm
- net Net-(D14-A): track 0.00 -> 1.43 mm
- net Net-(D10-A): track 0.00 -> 1.39 mm
- net Net-(D12-A): track 0.00 -> 1.37 mm
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
Commit message: update
Parts:
- moved G*** 0.42 mm to (133.5, 84.4)
Changed lines of the file:
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@@
 	(footprint "LOGO"
 		(layer "F.Cu")
-		(at 133.8 84.7)
+		(at 133.5 84.4)
 		(property "Reference" "G***"
 			(at 0 0 0)
@@
 			(at 0 1.43 180)
 			(layer "B.SilkS")
+			(hide yes)
 			(effects
 				(font
@@
 			(at 0 1.17 0)
 			(layer "B.SilkS")
+			(hide yes)
 			(effects
 				(font
@@
 			(at 0 2.83 0)
 			(layer "B.SilkS")
+			(hide yes)
 			(effects
 				(font
@@
 			(at 0 1.17 0)
 			(layer "B.SilkS")
+			(hide yes)
 			(effects
 				(font
@@
 			(at 0 1.17 180)
 			(layer "B.SilkS")
+			(hide yes)
 			(effects
 				(font
@@
 			(at 0 1.17 180)
 			(layer "B.SilkS")
+			(hide yes)
 			(effects
 				(font
@@
 			(at 0 1.17 0)
 			(layer "B.SilkS")
+			(hide yes)
 			(effects
 				(font
@@
 			(at 0 1.43 180)
 			(layer "B.SilkS")
+			(hide yes)
 			(effects
 				(font
@@
 			(at 0 1.17 180)
 			(layer "B.SilkS")
+			(hide yes)
 			(effects
 				(font
@@
 			(at 0 1.43 180)
 			(layer "B.SilkS")
+			(hide yes)
 			(effects
 				(font
@@
 			(at 0 1.17 180)
 			(layer "B.SilkS")
+			(hide yes)
 			(effects
 				(font
@@
 			(at 0 1.43 180)
 			(layer "B.SilkS")
+			(hide yes)
 			(effects
 				(font
@@
 			(at 0 1.43 180)
 			(layer "B.SilkS")
+			(hide yes)
 			(effects
 				(font
@@
 			(at 0 1.43 180)
 			(layer "B.SilkS")
+			(hide yes)
 			(effects
 				(font
@@
 			(at 0 1.16 0)
 			(layer "B.SilkS")
+			(hide yes)
 			(effects
 				(font
@@
 			(at 0 1.43 180)
 			(layer "B.SilkS")
+			(hide yes)
 			(effects
 				(font
@@
 			(at 0 1.17 180)
 			(layer "B.SilkS")
+			(hide yes)
 			(effects
 				(font

Commit message: update
Parts:
- removed the G*** at (139.4, 111.1)
- removed the G*** at (133.5, 84.4)
- removed the G*** at (155.8, 112.3)
- removed the G*** at (157.5, 92.2)
- removed the G*** at (151.7, 83.1)
- removed the G*** at (154.2, 96.0)
- removed the G*** at (129.2, 90.8)
- removed the G*** at (154.5, 84.7)
- removed the G*** at (144.2, 95.8)
- removed the G*** at (147.6, 107.9)
- removed the G*** at (154.3, 111.2)
- removed the G*** at (135.3, 108.9)
- removed the G*** at (130.4, 94.3)
- removed the G*** at (152.2, 98.8)
- removed the G*** at (137.1, 107.6)
- removed the G*** at (131.9, 91.9)
- added G***: LOGO, LOGO, F.Cu at (144.3, 96.8)
- added G***: LOGO, LOGO, F.Cu at (144.8, 96.6)
- D1, R2: moved to B.Cu
- moved R3 32.4 mm to (139.8, 110.5), turned to -20 degrees
- moved R6 31.5 mm to (158.7, 90.7), turned to -60 degrees
- moved D2 30.6 mm to (140.2, 109.4), turned to -20 degrees
- moved R2 30.1 mm to (155.1, 100.4)
- moved D5 29.9 mm to (157.7, 91.3), turned to -60 degrees
- moved R4 28.1 mm to (131.2, 103.0), turned to -60 degrees
- moved D3 27.4 mm to (132.5, 102.4), turned to -60 degrees
- moved R5 26.7 mm to (150.9, 82.6), turned to 160 degrees
- moved R8 25.9 mm to (131.2, 90.7), turned to 60 degrees
- moved D1 25.4 mm to (153.1, 100.5)
- moved D4 25.2 mm to (150.4, 83.7), turned to 160 degrees
- moved D7 22.3 mm to (132.2, 91.4), turned to 60 degrees
- moved R10 18.5 mm to (158.0, 102.5), turned to 60 degrees
- moved D9 17.7 mm to (156.8, 101.8), turned to 60 degrees
- moved R7 4.31 mm to (150.3, 110.1), turned to 30 degrees
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Routing:
- net +3.7V: track 175.7 -> 160.7 mm, vias 8 -> 22
- net GND: track 10.3 -> 16.3 mm, vias 19 -> 27
- net Net-(D1-A): track 4.25 -> 1.49 mm
- net /SWIO: track 16.4 -> 14.4 mm
- net /LED_DOUT: track 67.7 -> 68.3 mm, vias 1 -> 2
- net Net-(D7-A): track 1.89 -> 1.34 mm
