File: INNER_PCB/.history/INNER_PCB.kicad_pcb (KiCad board)
At the start: 2 copper layers, 50 x 50 mm, 82 parts, among them J1 Conn_01x03, J2 Conn_01x02, U2 CH32V003FxUx

Commit message: more art
Parts:
- removed the G*** at (130.5, 98.2)
Changed lines of the file:
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@@
-	(footprint "LOGO"
-		(layer "F.Cu")
-		(at 130.5 98.2)
-		(property "Reference" "G***"
-			(at 0 0 0)
-			(layer "F.SilkS")
-			(hide yes)
-			(effects
-				(font
-					(size 1.5 1.5)
-					(thickness 0.3)
-				)
-			)
-		)
-		(property "Value" "LOGO"
-			(at 0.75 0 0)
-			(layer "F.SilkS")
-			(hide yes)
-			(effects
-				(font
-					(size 1.5 1.5)
-					(thickness 0.3)
-				)
-			)
-		)
-		(property "Datasheet" ""
-			(at 0 0 0)
-			(layer "F.Fab")
-			(hide yes)
-			(effects
-				(font
-					(size 1.27 1.27)
-				)
-			)
-		)
-		(property "Description" ""
-			(at 0 0 0)
-			(layer "F.Fab")
-			(hide yes)
-			(effects
-				(font
-					(size 1.27 1.27)
-				)
-			)
-		)
-		(attr board_only exclude_from_pos_files exclude_from_bom)
-		(duplicate_pad_numbers_are_jumpers no)
-		(fp_poly
-			(pts
-				(xy 0.087395 -0.490718) (xy 0.171643 -0.465214) (xy 0.252682 -0.425391) (xy 0.325452 -0.373474)
-				(xy 0.355 -0.345893) (xy 0.416426 -0.270338) (xy 0.460114 -0.186623) (xy 0.485508 -0.101737) (xy 0.496348 -0.038002)
-				(xy 0.498653 0.016882) (xy 0.492398 0.072162) (xy 0.484944 0.107602) (xy 0.453667 0.199999) (xy 0.406975 0.282435)
-				(xy 0.347023 0.353551) (xy 0.275965 0.411987) (xy 0.195955 0.456384) (xy 0.109147 0.485382) (xy 0.017694 0.497622)
-				(xy -0.076249 0.491745) (xy -0.112184 0.48447) (xy -0.196373 0.455174) (xy -0.275975 0.41062) (xy -0.347075 0.353862)
-				(xy -0.405754 0.287951) (xy -0.443182 0.22651) (xy -0.465771 0.170138) (xy -0.484135 0.10569) (xy -0.496119 0.041996)
-				(xy -0.499679 -0.005) (xy -0.490401 -0.089403) (xy -0.464053 -0.17406) (xy -0.423028 -0.255136)
-				(xy -0.369717 -0.328791) (xy -0.306514 -0.391191) (xy -0.235811 -0.438496) (xy -0.226511 -0.443182)
-				(xy -0.170139 -0.465771) (xy -0.105691 -0.484135) (xy -0.041997 -0.496119) (xy 0.005 -0.499679)
-			)
-			(stroke
-				(width 0)
-				(type solid)
-			)
-			(fill yes)
-			(layer "F.SilkS")
-		)
-		(embedded_fonts no)
-	)
 	(footprint "LOGO"
 		(layer "F.Cu")
